File: esp32-s3-rf-board.kicad_sch (KiCad schematic)
At the start: 0 parts

Commit message: v1.2: 40 MHz crystal, ESP32-S3FN8 flash, real schematic
Closes the three fab-blockers for the bare QFN56 design. Adds Y1
(40 MHz NX3225GA) with C12/C13 12 pF NP0 load caps on XTAL_P/XTAL_N,
swaps U1 to ESP32-S3FN8 (8 MB internal flash, same QFN56 footprint),
and replaces the placeholder .kicad_sch with real symbols + nets
(ERC: 0 errors). Also adds EN 10k pull-up (R5), USB 22R series damping
(R6, R7), decaps repositioned within 2 mm of every VDD pad, and the
previously-uncommitted v1.1 USB-C CC / ESD / test-point work in
reroute_clean.py.

Layout cleanup still pending: the auto-generator leaves 135 DRC
violations and 122 unconnected nets (USB-C pads overlapping J5, LDO
near C8, RF keepout around antenna). Manual Pcbnew pass required
before sending Gerbers to JLCPCB.
Parts:
- added ANT1: 2450AT18A100, ANT_0402_1x0.5mm, symbol custom:ANT_CHIP_2P
- added C1, C10, C11, C2, C3, C4, C5, C6, C9: 100nF, C_0402, symbol custom:C
- added C12, C13: 12pF, C_0402, symbol custom:C
- added C7, C8: 10uF, C_0805, symbol custom:C_Bulk
- added D1: LED_RED, LED_0402, symbol custom:LED
- added D2: LED_GRN, LED_0402, symbol custom:LED
- added J1: USB_C_16P, USB-C_SMD_16P, symbol custom:USB_C_16P
- added J2: U.FL_SMD, U.FL_SMD, symbol custom:UFL_SMD
- added J3, J4: 1x04_2.54mm, PinHeader_1x04_P2.54mm, symbol custom:Header_1x04
- added J5: 1x06_2.54mm, PinHeader_1x06_P2.54mm, symbol custom:Header_1x06
- added R1: 330R, R_0402, symbol custom:R
- added R2: 1k, R_0402, symbol custom:R
- added R3, R4: 5.1k, R_0402, symbol custom:R
- added R5: 10k, R_0402, symbol custom:R
- added R6, R7: 22R, R_0402, symbol custom:R
- added SW1, SW2: SW_TACT_6x6, SW_Tactile_6x6mm, symbol custom:SW_Tactile
- added TP1: TP_3V3, TP_SMD_1.5mm, symbol custom:TestPoint_SMD
- added TP2: TP_GND, TP_SMD_1.5mm, symbol custom:TestPoint_SMD
- added TP3: TP_RF, TP_SMD_1.5mm, symbol custom:TestPoint_SMD
- added U1: ESP32-S3FN8, QFN-56_7x7mm_P0.4mm, symbol custom:ESP32-S3FN8
- added U2: AP2112K-3.3, SOT-23-5, symbol custom:AP2112K-3.3
- added U3: CP2102-GMR, QFN-28_5x5mm_P0.5mm, symbol custom:CP2102
- added U4: USBLC6-2SC6, SOT-23-6, symbol custom:USBLC6-2SC6
- added Y1: 40MHz_NX3225GA, XTAL_SMD_3225_4P, symbol custom:XTAL_3225_4P
Connections:
- new net 3V3: C1.1, C11.1, C2.1, C3.1, C4.1, C5.1, C6.1, C8.1, J3.2, J4.2, J5.2, R2.1, R5.1, TP1.1 (TP), U1.29 (VDD_SPI), U1.7 (VDD3P3), U1.8 (VDD3P3), U2.1 (EN), U2.5 (VOUT), U3.15 (VDD), U3.4 (VDD)
- new net 5V: C10.1, C7.1, C9.1, J1.A4 (VBUS), J1.A9 (VBUS), J1.B4 (VBUS), J1.B9 (VBUS), U2.3 (VIN), U4.5 (VBUS)
- new net EN: R5.2, SW1.3 (B), SW1.4 (B), U1.51 (CHIP_PU)
- new net GND: ANT1.2 (GND), C1.2, C10.2, C11.2, C12.2, C13.2, C2.2, C3.2, C4.2, C5.2, C6.2, C7.2, C8.2, C9.2, D1.2, D2.2, J1.A1 (GND), J1.A12 (GND), J1.B1 (GND), J1.B12 (GND), J1.S1 (SHIELD), J2.2 (GND), J2.3 (GND), J3.1, J4.1, J5.1, R3.2, R4.2, SW1.1 (A), SW1.2 (A), SW2.1 (A), SW2.2 (A), TP2.1 (TP), U1.1 (GND), U1.15 (GND), U1.4 (GND), U1.43 (GND), U1.56 (GND), U1.57 (EP/GND), U2.2 (GND), U3.1 (GND), U3.16 (GND), U3.22 (GND), U3.29 (EP), U3.8 (GND), U4.2 (GND), Y1.2 (GND), Y1.4 (GND)
- new net GPIO0: SW2.3 (B), SW2.4 (B), U1.52 (IO0)
- new net GPIO48_LED: R1.1, U1.48 (IO48/LED)
- new net I2C_SCL: J4.4, U1.23 (IO9/SCL)
- new net I2C_SDA: J4.3, U1.22 (IO8/SDA)
- new net LED_POWER_A: D2.1, R2.2
- new net LED_STATUS_A: D1.1, R1.2
- new net RF_ANT: ANT1.1 (RF), J2.1 (SIG), TP3.1 (TP), U1.36 (LNA_IN)
- new net SPI_CS: J5.6, U1.19 (IO10/CS)
- new net SPI_MISO: J5.4, U1.17 (IO13/MISO)
- new net SPI_MOSI: J5.3, U1.16 (IO11/MOSI)
- new net SPI_SCK: J5.5, U1.18 (IO12/CLK)
- new net UART_RX: J3.4, U1.21 (IO44/RXD0), U3.10 (RXD)
- new net UART_TX: J3.3, U1.20 (IO43/TXD0), U3.9 (TXD)
- new net USB_CC1: J1.A5 (CC1), R3.1
- new net USB_CC2: J1.B5 (CC2), R4.1
- new net USB_DM: J1.A7 (D-), J1.B7 (D-), R7.2, U4.1 (I/O1), U4.6 (I/O1)
- new net USB_DM_CP: R7.1, U3.2 (D-)
- new net USB_DP: J1.A6 (D+), J1.B6 (D+), R6.2, U4.3 (I/O2), U4.4 (I/O2)
- new net USB_DP_CP: R6.1, U3.3 (D+)
- new net XTAL_N: C13.1, U1.40 (XTAL_N), Y1.3 (XO)
- new net XTAL_P: C12.1, U1.39 (XTAL_P), Y1.1 (XI)
Other:
- note added: "ESP32-S3 RF Dev Board v1.2 -- schematic generated by generate_board.py"
- note added: "Power tree: USB-C 5V -> USBLC6 (ESD) -> AP2112K-3.3 LDO -> 3V3 rail. Note: AP2112K EN is tied to VIN to keep LDO always on when power is applied."
- note added: "RF: 50-ohm microstrip from ESP32 LNA_IN to chip antenna (ANT1). Load caps C12/C13 = 12 pF NP0 (CL ~ 8-10 pF; crystal datasheet CL nominal 8 pF)."
- note added: "Strapping pins at boot: IO0 must be HIGH -- SW2 pulls low to enter download mode IO45 / IO46 -- leave at default (SPI boot + voltage select)"
- note removed: "- 50-ohm microstrip: 0.6mm wide on F.Cu, 0.2mm prepreg (7628) to In1.Cu GND plane - Keepout zone: 5mm radius around ANT1, no copper any layer - GND stitching vias: every 6mm along RF trace (lambda/10 at 2.4GHz in FR4) - Er=4.4 (7628 prepreg), loss tangent=0.02"
- note removed: "ESP32-S3 RF Development Board - Schematic Placeholder"
- note removed: "Power Tree: USB-C VBUS (5V) -> C9,C10 bypass -> AP2112K-3.3 LDO -> C7(in),C8(out) -> 3.3V rail 3.3V -> ESP32-S3 (C1-C6 decoupling) | CP2102 (C11) | LED (R2,D2)"
- note removed: "RF Design Notes:"
- note removed: "See PCB layout for full design. Component list: U1: ESP32-S3 QFN56 U2: AP2112K-3.3V SOT-23-5 U3: CP2102-GMR QFN-28 ANT1: Johanson 2450AT18A100 J1: USB-C 16P J2: u.FL connector J3: UART 4-pin header J4: I2C 4-pin header J5: SPI 6-pin header SW1: Reset button SW2: Boot button D1: Status LED (red) D2: Power LED (green) R1: 330R (status LED) R2: 1k (power LED) C1-C6: 100nF decoupling (ESP32-S3) C7-C8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"
